Commit message: update urdf and docs

File: aifred_description/urdf/aifred.urdf.xacro (robot description, xacro)
@@ -229,5 +229,6 @@
        The head meshes were exported from CAD with an arbitrary origin, so the head
        is placed by putting the back face of its mounting plate (CAD x = 0.15997,
-       centered at y = 0.005692, z = 0.400532) at head_mount_x along wrist_link's x axis. -->
+       centered at y = 0.005692, z = 0.400532) at head_mount_x along wrist_link's x axis.
+       head_mount_link's frame sits at that point; its mesh is offset back by the CAD coordinates. -->
   <xacro:property name="head_mount_x" value="0.065"/>
   <xacro:property name="head_mesh_dir" value="package://interbotix_xsarm_descriptions/meshes/aifred_meshes"/>
@@ -236,5 +237,5 @@
   </material>
   <joint name="head_mount" type="fixed">
-    <origin rpy="0 0 0" xyz="${head_mount_x - 0.15997} -0.005692 -0.400532"/>
+    <origin rpy="0 0 0" xyz="${head_mount_x} 0 0"/>
     <parent link="$(arg robot_name)/wrist_link"/>
     <child link="$(arg robot_name)/head_mount_link"/>
@@ -242,5 +243,5 @@
   <link name="$(arg robot_name)/head_mount_link">
     <visual>
-      <origin rpy="0 0 0" xyz="0 0 0"/>
+      <origin rpy="0 0 0" xyz="-0.15997 -0.005692 -0.400532"/>
       <geometry>
         <mesh filename="${head_mesh_dir}/base_link.stl" scale="0.001 0.001 0.001"/>
@@ -249,5 +250,5 @@
     </visual>
     <collision>
-      <origin rpy="0 0 0" xyz="0 0 0"/>
+      <origin rpy="0 0 0" xyz="-0.15997 -0.005692 -0.400532"/>
       <geometry>
         <mesh filename="${head_mesh_dir}/base_link.stl" scale="0.001 0.001 0.001"/>
@@ -255,5 +256,5 @@
     </collision>
     <inertial>
-      <origin rpy="0 0 0" xyz="0.16147000792413785 0.005693053609813656 0.4003205773306801"/>
+      <origin rpy="0 0 0" xyz="0.00150000792413785 0.000001053609813656 -0.0002114226693199"/>
       <mass value="0.03498801320160599"/>
       <inertia ixx="9e-06" iyy="5e-06" izz="5e-06" ixy="0" iyz="0" ixz="0"/>
@@ -261,5 +262,5 @@
   </link>
   <joint name="head_base_joint" type="fixed">
-    <origin rpy="0 0 0" xyz="0.16297 0.005692 0.400532"/>
+    <origin rpy="0 0 0" xyz="0.003 0 0"/>
     <parent link="$(arg robot_name)/head_mount_link"/>
     <child link="$(arg robot_name)/head_link"/>

Commit message: improve robot model and poses

File: aifred_description/urdf/aifred.urdf.xacro (robot description, xacro)
@@ -226,5 +226,5 @@
     </inertial>
   </link>
-  <!-- AIfred head: replaces the wrist_rotate motor and the gripper.
+  <!-- AIfred head: replaces the gripper and is mounted on the wrist_rotate motor horn.
        The head meshes were exported from CAD with an arbitrary origin, so the head
        is placed by putting the back face of its mounting plate (CAD x = 0.15997,
@@ -236,9 +236,21 @@
     <color rgba="0.700 0.700 0.700 1.000"/>
   </material>
-  <joint name="head_mount" type="fixed">
+  <joint name="wrist_rotate" type="revolute">
+    <axis xyz="1 0 0"/>
+    <limit effort="1" lower="${-pi}" upper="${pi}" velocity="${pi}"/>
     <origin rpy="0 0 0" xyz="${head_mount_x} 0 0"/>
     <parent link="$(arg robot_name)/wrist_link"/>
     <child link="$(arg robot_name)/head_mount_link"/>
-  </joint>
+    <dynamics friction="0.1"/>
+  </joint>
+  <transmission name="trans_wrist_rotate">
+    <type>transmission_interface/SimpleTransmission</type>
+    <joint name="wrist_rotate">
+      <hardwareInterface>hardware_interface/EffortJointInterface</hardwareInterface>
+    </joint>
+    <actuator name="wrist_rotate_motor">
+      <mechanicalReduction>1</mechanicalReduction>
+    </actuator>
+  </transmission>
   <link name="$(arg robot_name)/head_mount_link">
     <visual>
@@ -330,4 +342,13 @@
     </inertial>
   </link>
+  <!-- End-effector frame for the Python API (M in mr_descriptions.py): same point as camera_link,
+       aligned with base_link at the home pose (x forward, y left, z up), like a gripper.
+       The lens looks out along -z, so roll = pitch = 0 keeps the camera parallel to the floor. -->
+  <joint name="ee_camera_joint" type="fixed">
+    <origin rpy="0 0 0" xyz="0 0 0"/>
+    <parent link="$(arg robot_name)/camera_link"/>
+    <child link="$(arg robot_name)/ee_camera_link"/>
+  </joint>
+  <link name="$(arg robot_name)/ee_camera_link"/>
   <joint name="projector_joint" type="fixed">
     <origin rpy="0 0 0" xyz="0.027243 -0.007585 0.00745"/>
